Commit message: 添加 EKF 融合定位：引入 robot_localization 节点，融合 Wheel Odometry 和 IMU 数据，生成 /odometry/filtered 话题，有效解决了麦轮小车在仿真/真机中因打滑导致的里程计漂移问题。

File: mbot_description/urdf/mbot.urdf.xacro (robot description, xacro)
@@ -107,4 +107,5 @@
 <!-- 插件 -->
 <xacro:lidar_plugin frame_prefix="lidar_link" min_angle="${safe_min_angle}" max_angle="${safe_max_angle}" />
+<xacro:imu_plugin frame_prefix="imu_center_link"/>
 <xacro:mbot_ros2_control name="MbotSystem" use_sim="$(arg use_sim)"/>
 </robot>

File: mbot_description/urdf/plugin/gazebo_sensor_plugin.xacro (robot description, xacro)
@@ -38,3 +38,61 @@
         </gazebo>
     </xacro:macro>
+    <xacro:macro name="imu_plugin" params="frame_prefix">
+        <gazebo reference="${frame_prefix}">
+            <gravity>true</gravity>
+            <sensor name="imu_sensor" type="imu">
+            <always_on>true</always_on>
+            <update_rate>100</update_rate> <visualize>true</visualize>
+            <topic>__default_topic__</topic>
+            <plugin filename="libgazebo_ros_imu_sensor.so" name="imu_plugin">
+                <ros>
+                <remapping>~/out:=/imu/data</remapping>
+                </ros>
+                <initial_orientation_as_reference>false</initial_orientation_as_reference>
+            </plugin>
+            <imu>
+                <angular_velocity>
+                <x>
+                    <noise type="gaussian">
+                    <mean>0.0</mean>
+                    <stddev>2e-4</stddev>
+                    </noise>
+                </x>
+                <y>
+                    <noise type="gaussian">
+                    <mean>0.0</mean>
+                    <stddev>2e-4</stddev>
+                    </noise>
+                </y>
+                <z>
+                    <noise type="gaussian">
+                    <mean>0.0</mean>
+                    <stddev>2e-4</stddev>
+                    </noise>
+                </z>
+                </angular_velocity>
+                <linear_acceleration>
+                <x>
+                    <noise type="gaussian">
+                    <mean>0.0</mean>
+                    <stddev>1.7e-2</stddev>
+                    </noise>
+                </x>
+                <y>
+                    <noise type="gaussian">
+                    <mean>0.0</mean>
+                    <stddev>1.7e-2</stddev>
+                    </noise>
+                </y>
+                <z>
+                    <noise type="gaussian">
+                    <mean>0.0</mean>
+                    <stddev>1.7e-2</stddev>
+                    </noise>
+                </z>
+                </linear_acceleration>
+            </imu>
+            </sensor>
+        </gazebo>
+    </xacro:macro>
 </robot>
